File: dumbesc_hw.kicad_sch (KiCad schematic)
At the start: 39 parts

Commit message: finish schematic
Parts:
- removed C? (x2): 0.1uF, Capacitor_SMD:C_0603_1608Metric, symbol Device:C
- removed D?: GREEN, LED_SMD:LED_0402_1005Metric, symbol Device:LED
- removed D?: 1PS79SB30, Diode_SMD:D_SOD-523, symbol Device:D_Schottky
- removed Q? (x6): 2N7002, Package_TO_SOT_SMD:SOT-23, symbol Transistor_FET:2N7002
- removed R?: 470, Resistor_SMD:R_0402_1005Metric, symbol Device:R
- removed U?: TLV71333PDQN, Package_SON:Texas_X2SON-4_1x1mm_P0.65mm, symbol TLV71333PDQ:TLV71333PDQN
- added C?: 0.1uF, symbol Device:C
- added C?: 1uF, symbol Device:C
- added D? (x2): LED, symbol Device:LED
- added R? (x2): 1K, symbol Device:R
- added R?: 10K, symbol Device:R
- added U?: ADS1018IDGS, symbol Analog_ADC:ADS1018IDGS
Connections:
- net +3V3: now also C?.1, C?.2, U?.8 (VDD)
- net GND: now also C?.1, C?.2, R?.2, R?.2, R?.2, U?.3 (GND)
- net CAN_SILENT: now reaches U?.11 (GPIO8)
- net PWM_INPUT: now reaches U?.12 (GPIO9)
- net SPI1_SCK: now reaches U?.14 (GPIO11)
- net SPI1_SCK: now also U?.1 (SCLK)
- net SPI1_PICO: now reaches U?.15 (GPIO12)
- net SPI1_PICO: now also U?.10 (DIN)
- net SPI1_POCI: now reaches U?.16 (GPIO13)
- net SPI1_POCI: now also U?.9 (DOUT/~{DRDY})
- net SPI1_nCS: now reaches U?.17 (GPIO14)
- net SPI1_nCS: now also U?.2 (~{CS})
- net PWM0A_HINA: now reaches U?.2 (GPIO0)
- net UART0_TX_DEBUG: now reaches U?.27 (GPIO16)
- net UART0_RX_DEBUG: now reaches U?.28 (GPIO17)
- net USB_VBUS: now reaches U?.29 (GPIO18)
- net PWM0B_LINA: now reaches U?.3 (GPIO1)
- net LED0: now reaches U?.30 (GPIO19)
- net LED0: now also D?.2 (A)
- net LED1: now reaches U?.31 (GPIO20)
- net LED1: now also D?.2 (A)
- net VSENSE_BATT: now reaches U?.38 (GPIO26_ADC0)
- net VSENSE_A: now reaches U?.39 (GPIO27_ADC1)
- net PWM1A_HINB: now reaches U?.4 (GPIO2)
- net VSENSE_B: now reaches U?.40 (GPIO28_ADC2)
- net VSENSE_C: now reaches U?.41 (GPIO29_ADC3)
- net PWM1B_LINB: now reaches U?.5 (GPIO3)
- net PWM2A_HINC: now reaches U?.6 (GPIO4)
- net PWM2B_LINC: now reaches U?.7 (GPIO5)
- net PIO0_CAN_TX: now reaches U?.8 (GPIO6)
- net PIO0_CAN_RX: now reaches U?.9 (GPIO7)
- new net: D?.1 (K), R?.1 (x2)
- new net: R?.1, U?.7 (AIN3)
- new net ISENSE_A: U?.4 (AIN0)
- new net ISENSE_B: U?.5 (AIN1)
- new net ISENSE_C: U?.6 (AIN2)
- no-connect marks 3 -> 7
Other:
- added sheet Drive Stage (drive.kicad_sch)
- added sheet Interfaces (interfaces.kicad_sch)
- added sheet Power Stage (power.kicad_sch)
- note removed: "3V3 Regulation"
- moved on the sheet: R?, TP?
